File: KiCad/Amp Module.sch (KiCad schematic (older format))
At the start: 9 parts

Commit message: Update schematics
Parts:
- removed J?: IDC34, symbol Connector_Generic:Conn_02x17_Odd_Even
- added D? (x3): LED_Small, symbol Device:LED_Small
- added J?: IDC34, symbol Connector_Generic:Conn_02x17_Odd_Even
- added Q?: Q_PNP, symbol Device:Q_PNP_BCE
- added R? (x3): R_Small, symbol Device:R_Small
- added R?: 100k, symbol Device:R_Small
- added SW?: MUTE_BUTTON, symbol Switch:SW_SPST
Connections:
- net labels added: +12VDCOUT, +5VDCOUT, +VCCMON, -12VDCOUT, -VCCMON, LM_+5VDCOUT, LM_IOUT1MON, LM_IOUT2MON, LM_IOUT3MON, LM_IOUT4MON, LM_MUTE1, LM_MUTE2, LM_MUTE3, LM_MUTE4, LM_PROTECT1, LM_PROTECT2, LM_PROTECT3, LM_PROTECT4, LM_READY1, LM_READY2, LM_READY3, LM_READY4, LM_TEMPMON12, LM_TEMPMON34, LM_VOUT1MON, LM_VOUT2MON, LM_VOUT3MON, LM_VOUT4MON, RESERVED_A, RESERVED_A2, RESERVED_B, SDPWS
- net labels removed: DSP_+VCCMON, DSP_-VCCMON
- wire segments 28 -> 67
- no-connect marks 6 -> 0
Other:
- note added: "DSP IDC"
- note added: "MUTE"
- note added: "MUTE_SIGNAL"
- note added: "PROTECTION"
- note added: "PROTECT_SIGNAL"
- note added: "READY1/3"
- note added: "READY2/4"
- note added: "SBAGLIATO"
- moved on the sheet: J?, R?, RV?

Commit message: Update schematic
Parts:
- removed D? (x2): LED_Small, symbol Device:LED_Small
- removed R? (x2): R_Small, symbol Device:R_Small
- removed R?: 100k, symbol Device:R_Small
- added D? (x3): LED_Small, symbol Device:LED_Small
- added Q?: PNP, symbol Device:Q_PNP_BCE
- added Q? (x2): NPN, symbol Device:Q_NPN_BCE
- added R?: 100k, symbol Device:R_Small
- added R? (x3): R_Small, symbol Device:R_Small
- added R? (x3): 10k, symbol Device:R_Small
- added SW?: MUTE_BUTTON, symbol Switch:SW_SPST
- added U? (x5): 74LS32, symbol 74xx:74LS32
- Q?: value Q_PNP -> PNP
- R?: value R_Small -> 150
Connections:
- net labels added: +12VDC, +5VDC, -12VDC, DSP_MUTE1, DSP_MUTE2
- net labels removed: +12VDCOUT, -12VDCOUT, DSP_+12VDCIN, DSP_-12VDCIN, DSP_MUTE, LM_+5VDCOUT
- wire segments 67 -> 90
Other:
- note added: "LITEMOD IDC"
- note added: "sbagliato cazzo"
- note removed: "MUTE_SIGNAL"
- note removed: "PROTECT_SIGNAL"
- note removed: "SBAGLIATO"
- moved on the sheet: D?, J?, Q?, R?, RV?

Commit message: Update schematic
Parts:
- removed D? (x2): LED_Small, symbol Device:LED_Small
- removed Q?: PNP, symbol Device:Q_PNP_BCE
- removed R?: 100k, symbol Device:R_Small
- removed R?: R_Small, symbol Device:R_Small
- removed SW?: MUTE_BUTTON, symbol Switch:SW_SPST
- added D? (x3): LED_Small, symbol Device:LED_Small
- added Q?: NPN, symbol Device:Q_NPN_BCE
- added Q? (x3): PNP, symbol Device:Q_PNP_BCE
- added R? (x5): R_Small, symbol Device:R_Small
- added R?: ?, symbol Device:R_Small
- added R?: 150, symbol Device:R_Small
- added R?: 10k, symbol Device:R_Small
- added SW?: MUTE_BUTTON, symbol Switch:SW_SPST
- added U? (x2): 74LVC2G08, symbol 74xGxx:74LVC2G08
Connections:
- net labels added: DSP_READY13, DSP_READY24, LM_IN1+, LM_IN1-, LM_IN2+, LM_IN2-, LM_IN3+, LM_IN3-, LM_IN4+, LM_IN4-
- net labels removed: SIG_1+, SIG_1-, SIG_2+, SIG_2-
- wire segments 90 -> 121
Other:
- note added: "Protection 1 signal"
- note added: "READY"
- note added: "TODO:\n - Voltage output monitor\n - Protection alert LEDs"
- note added: "VOLUME CONTROL"
- note removed: "READY1/3"
- note removed: "sbagliato cazzo"
- moved on the sheet: D?, J?, Q?, R?, RV?

Commit message: Update schematic
Parts:
- removed D? (x2): LED_Small, symbol Device:LED_Small
- removed Q? (x2): NPN, symbol Device:Q_NPN_BCE
- removed R? (x2): 10k, symbol Device:R_Small
- removed R? (x2): R_Small, symbol Device:R_Small
- removed U? (x2): 74LS32, symbol 74xx:74LS32
Connections:
- wire segments 121 -> 105
Other:
- note removed: "PROTECTION"
Changed lines of the file:
@@
 	5100 2300 5100 2200
-Wire Notes Line
-	8100 600  8100 2850
-Wire Notes Line
-	8100 2850 11100 2850
-Wire Notes Line
-	11100 2850 11100 600
-Wire Notes Line
-	11100 600  8100 600
-Text Notes 8100 700  0    50   ~ 0
-PROTECTION
 Wire Notes Line
 	2900 600  2900 2850
@@
 Wire Notes Line
 	3100 700  3100 600
-Wire Notes Line
-	8100 700  8600 700
-Wire Notes Line
-	8600 700  8600 600
 Wire Notes Line
 	2800 600  2800 2850
@@
 Text GLabel 3650 1150 0    50   Input ~ 0
 DSP_MUTE1
-Text GLabel 9850 900  0    50   Input ~ 0
-+5VDC
 Text GLabel 1450 1550 0    50   Input ~ 0
 +12VDC
@@
 Text GLabel 1950 1950 2    50   Input ~ 0
 +12VDC
-Text GLabel 8750 1250 0    50   Input ~ 0
-LM_PROTECT1
-Text GLabel 8750 1450 0    50   Input ~ 0
-LM_PROTECT3
-Text GLabel 8750 2500 0    50   Input ~ 0
-LM_PROTECT4
-Text GLabel 8750 2300 0    50   Input ~ 0
-LM_PROTECT2
-Text GLabel 8800 1650 0    50   Input ~ 0
-DSP_PROTECT1
-Text GLabel 8800 2700 0    50   Input ~ 0
-DSP_PROTECT2
-$Comp
-L Device:R_Small R?
-U 1 1 5FD513D9
-P 9700 1350
-F 0 "R?" V 9504 1350 50  0000 C CNN
-F 1 "10k" V 9595 1350 50  0000 C CNN
-F 2 "" H 9700 1350 50  0001 C CNN
-F 3 "~" H 9700 1350 50  0001 C CNN
-	1    9700 1350
-	0    1    1    0
-$EndComp
-$Comp
-L Device:Q_NPN_BCE Q?
-U 1 1 5FD53EF6
-P 10150 1350
-F 0 "Q?" H 10341 1396 50  0000 L CNN
-F 1 "NPN" H 10341 1305 50  0000 L CNN
-F 2 "" H 10350 1450 50  0001 C CNN
-F 3 "~" H 10150 1350 50  0001 C CNN
-	1    10150 1350
-	1    0    0    -1
-$EndComp
-Wire Wire Line
-	9950 1350 9800 1350
-Text GLabel 9800 1950 0    50   Input ~ 0
-+5VDC
-Wire Wire Line
-	9400 2400 9350 2400
-$Comp
-L Device:R_Small R?
-U 1 1 5FD699D4
-P 9700 2400
-F 0 "R?" V 9504 2400 50  0000 C CNN
-F 1 "10k" V 9595 2400 50  0000 C CNN
-F 2 "" H 9700 2400 50  0001 C CNN
-F 3 "~" H 9700 2400 50  0001 C CNN
-	1    9700 2400
-	0    1    1    0
-$EndComp
-Wire Wire Line
-	9600 2400 9400 2400
-Connection ~ 9400 2400
-$Comp
-L Device:Q_NPN_BCE Q?
-U 1 1 5FD6C7D3
-P 10150 2400
-F 0 "Q?" H 10341 2446 50  0000 L CNN
-F 1 "NPN" H 10341 2355 50  0000 L CNN
-F 2 "" H 10350 2500 50  0001 C CNN
-F 3 "~" H 10150 2400 50  0001 C CNN
-	1    10150 2400
-	1    0    0    -1
-$EndComp
-Wire Wire Line
-	9950 2400 9800 2400
-$Comp
-L Device:LED_Small D?
-U 1 1 5FD85142
-P 10250 1050
-F 0 "D?" V 10296 980 50  0000 R CNN
-F 1 "LED_Small" V 10205 980 50  0000 R CNN
-F 2 "" V 10250 1050 50  0001 C CNN
-F 3 "~" V 10250 1050 50  0001 C CNN
-	1    10250 1050
-	0    -1   -1   0
-$EndComp
-$Comp
-L Device:R_Small R?
-U 1 1 5FD868D0
-P 10050 900
-F 0 "R?" V 10246 900 50  0000 C CNN
-F 1 "R_Small" V 10150 900 50  0000 C CNN
-F 2 "" H 10050 900 50  0001 C CNN
-F 3 "~" H 10050 900 50  0001 C CNN
-	1    10050 900
-	0    -1   -1   0
-$EndComp
-$Comp
-L power:GND #PWR?
-U 1 1 5FD8F4A8
-P 10250 1550
-F 0 "#PWR?" H 10250 1300 50  0001 C CNN
-F 1 "GND" H 10255 1377 50  0000 C CNN
-F 2 "" H 10250 1550 50  0001 C CNN
-F 3 "" H 10250 1550 50  0001 C CNN
-	1    10250 1550
-	-1   0    0    -1
-$EndComp
-$Comp
-L power:GND #PWR?
-U 1 1 5FDAB89B
-P 10250 2600
-F 0 "#PWR?" H 10250 2350 50  0001 C CNN
-F 1 "GND" H 10255 2427 50  0000 C CNN
-F 2 "" H 10250 2600 50  0001 C CNN
-F 3 "" H 10250 2600 50  0001 C CNN
-	1    10250 2600
-	-1   0    0    -1
-$EndComp
-$Comp
-L Device:LED_Small D?
-U 1 1 5FDAC898
-P 10250 2100
-F 0 "D?" V 10296 2030 50  0000 R CNN
-F 1 "LED_Small" V 10205 2030 50  0000 R CNN
-F 2 "" V 10250 2100 50  0001 C CNN
-F 3 "~" V 10250 2100 50  0001 C CNN
-	1    10250 2100
-	0    -1   -1   0
-$EndComp
-$Comp
-L Device:R_Small R?
-U 1 1 5FDAC89E
-P 10050 1950
-F 0 "R?" V 10246 1950 50  0000 C CNN
-F 1 "R_Small" V 10155 1950 50  0000 C CNN
-F 2 "" H 10050 1950 50  0001 C CNN
-F 3 "~" H 10050 1950 50  0001 C CNN
-	1    10050 1950
-	0    -1   -1   0
-$EndComp
-$Comp
-L 74xx:74LS32 U?
-U 1 1 5FDB9273
-P 9050 1350
-F 0 "U?" H 9050 1675 50  0000 C CNN
-F 1 "74LS32" H 9050 1584 50  0000 C CNN
-F 2 "" H 9050 1350 50  0001 C CNN
-F 3 "http://www.ti.com/lit/gpn/sn74LS32" H 9050 1350 50  0001 C CNN
-	1    9050 1350
-	1    0    0    -1
-$EndComp
-$Comp
-L 74xx:74LS32 U?
-U 2 1 5FDBC748
-P 9050 2400
-F 0 "U?" H 9050 2725 50  0000 C CNN
-F 1 "74LS32" H 9050 2634 50  0000 C CNN
-F 2 "" H 9050 2400 50  0001 C CNN
-F 3 "http://www.ti.com/lit/gpn/sn74LS32" H 9050 2400 50  0001 C CNN
-	2    9050 2400
-	1    0    0    -1
-$EndComp
 $Comp
 L 74xx:74LS32 U?
@@
 	0    1    1    0
 $EndComp
-Wire Wire Line
-	9850 900  9950 900
-Wire Wire Line
-	9800 1950 9950 1950
-Wire Wire Line
-	10150 1950 10250 1950
-Wire Wire Line
-	10250 1950 10250 2000
-Wire Wire Line
-	10250 900  10250 950
-Wire Wire Line
-	10150 900  10250 900
-Wire Wire Line
-	9350 1350 9400 1350
-Wire Wire Line
-	9400 2700 8800 2700
-Wire Wire Line
-	9400 2400 9400 2700
-Wire Wire Line
-	9400 1350 9400 1650
-Wire Wire Line
-	9400 1650 8800 1650
-Connection ~ 9400 1350
-Wire Wire Line
-	9400 1350 9600 1350
 Wire Notes Line
 	600  5450 600  7700

Commit message: schematic updated
Parts:
- removed D? (x2): LED_Small, symbol Device:LED_Small
- removed Q?: NPN, symbol Device:Q_NPN_BCE
- removed Q? (x2): PNP, symbol Device:Q_PNP_BCE
- removed R? (x2): 12k, symbol Device:R_Small
- removed R? (x5): R_Small, symbol Device:R_Small
- removed R?: ?, symbol Device:R_Small
- removed R?: 150, symbol Device:R_Small
- removed RV?: 100k, symbol Device:R_POT_Dual
- added D?: LED_Small, symbol Device:LED_Small
- added R? (x4): ?, symbol Device:R_Small
- added R? (x2): 12k, symbol Device:R_Small
- added R?: 150, symbol Device:R_Small
- added RV?: 100k, symbol Device:R_POT_Dual
- gave numbers to parts that had none: 16
Connections:
- net labels removed: +5VDCOUT
- wire segments 105 -> 88
Other:
- note added: "TODO:\n - Voltage output monitor\n - Protection alert LEDs\n - Check volume impedance"
- note removed: "Protection 1 signal"
- note removed: "TODO:\n - Voltage output monitor\n - Protection alert LEDs"
- moved on the sheet: D1, J2, J3, Q1, Q5, R1, R13, R2, R5, R6, RV1

Commit message: schematic updated
Parts:
- removed D1, D?: LED_Small, symbol Device:LED_Small
- removed Q1, Q5: PNP, symbol Device:Q_PNP_BCE
- removed R13, R5: 10k, symbol Device:R_Small
- removed R6, R?: 150, symbol Device:R_Small
- removed SW1, SW2: MUTE_BUTTON, symbol Switch:SW_SPST
- removed U1: 74LVC2G08, symbol 74xGxx:74LVC2G08
- removed U2: 74LS32, symbol 74xx:74LS32
- added D? (x4): LED_Small, symbol Device:LED_Small
- added Q? (x4): S9012, symbol Device:Q_PNP_BCE
- added R? (x2): 100k, symbol Device:R_Small
- added R? (x4): 10k, symbol Device:R_Small
- added R? (x4): 150, symbol Device:R_Small
- added SW? (x2): SPDT, symbol Switch:SW_Push_SPDT
- added U? (x10): 74LS08, symbol 74xx:74LS08
Connections:
- net labels added: DSP_PROTECT13, DSP_PROTECT24
- net labels removed: DSP_PROTECT1, DSP_PROTECT2
- wire segments 88 -> 111
- no-connect marks 0 -> 6
Other:
- note added: "TODO:\n - Voltage output monitor\n - Check volume impedance"
- note removed: "MUTE"
- note removed: "READY"
- note removed: "READY2/4"
- note removed: "TODO:\n - Voltage output monitor\n - Protection alert LEDs\n - Check volume impedance"

Commit message: updated schematic
Parts:
- removed R?: ?, symbol Device:R_Small
- removed U? (x2): 74LS08, symbol 74xx:74LS08
- added D10, D11, D12, D5, D6, D7, D8, D9: LED_Small, symbol Device:LED_Small
- added R11: ?, symbol Device:R_Small
- added R19, R20, R21, R22, R23, R24, R25, R26, R27, R28: R_Small, symbol Device:R_Small
- added U3: CD4053B, symbol Analog_Switch:CD4053B
- added U4, U5, U6, U7, U8: LM393, symbol Comparator:LM393
- gave numbers to parts that had none: 28
- renumbered R1 to R4, R2 to R5
Connections:
- net DSP_SDPWS is gone; now on net SDPWS: J1.34 (Pin_34)
- net +5VDC: now also D10.2 (A), D11.2 (A), D12.2 (A), D5.2 (A), D6.2 (A), D7.2 (A), D8.2 (A), D9.2 (A), R19.1, R24.1, U3.16 (VDD), U4.8 (V+), U5.8 (V+), U6.8 (V+), U7.8 (V+), U8.8 (V+)
- net DSP_VOUT1MON: now also U3.14 (A), U5.2 (-), U5.6 (-), U6.2 (-), U6.6 (-)
- net DSP_VOUT2MON: now also U3.15 (B), U7.2 (-), U7.6 (-), U8.2 (-), U8.6 (-)
- net GND: now also R3.1, R11.1, R23.2, R28.2, U3.6 (INH), U3.7 (VEE), U3.8 (VSS), U4.4 (V-), U5.4 (V-), U6.4 (V-), U7.4 (V-), U8.4 (V-); no longer R3.2
- net LM_VOUT1MON: now also U3.12 (A0), U4.2 (-)
- net LM_VOUT2MON: now also U3.2 (B0), U4.6 (-)
- net LM_VOUT3MON: now also U3.13 (A1), U4.3 (+)
- net LM_VOUT4MON: now also U3.1 (B1), U4.5 (+)
- net RESERVED_A: no longer J2.3 (Pin_3), J3.3 (Pin_3)
- net RESERVED_A2: now also J3.3 (Pin_3); no longer J2.32 (Pin_32)
- net RESERVED_B: no longer J3.32 (Pin_32)
- net at RV1.6: now also R3.2; no longer R3.1
- net at RV2.6: now also R11.2
- new net: D9.1 (K), U7.1
- new net: R24.2, R25.1, U7.3 (+)
- new net: R25.2, R26.1, U7.5 (+)
- new net: D10.1 (K), U7.7
- new net: D11.1 (K), U8.1
- new net: R26.2, R27.1, U8.3 (+)
- new net: R27.2, R28.1, U8.5 (+)
- new net: D12.1 (K), U8.7
- new net: D5.1 (K), U5.1
- new net: R19.2, R20.1, U5.3 (+)
- new net: R20.2, R21.1, U5.5 (+)
- new net: D6.1 (K), U5.7
- new net: R22.2, R23.1, U6.5 (+)
- new net: D8.1 (K), U6.7
- new net: R21.2, R22.1, U6.3 (+)
- new net: D7.1 (K), U6.1
- new net RESERVED_A1: J2.3 (Pin_3)
- new net RESERVED_B1: J2.32 (Pin_32)
- new net RESERVED_B2: J3.32 (Pin_32)
- new net S1: U3.11 (S1), U4.1
- new net S2: U3.10 (S2), U4.7
- no-connect marks 6 -> 4
Other:
- note added: "MUTE"
- note added: "PROTECTION"
- note added: "READY"
- note added: "S1=0"
- note added: "S1=1"
- note added: "S2=0"
- note added: "S2=1"
- note added: "TODO:\n - Check volume impedance\n - Check protection high level voltage\n - Bypass caps\n - Decide about RESERVED pins"
- note added: "VOUT MONITOR"
- note removed: "TODO:\n - Voltage output monitor\n - Check volume impedance"
- moved on the sheet: D1, D2, D3, Q1, Q2, Q3, R10, R15, R16, R2, R3, R6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

Commit message: updated schematic to latest KiCad version
Parts:
- U4, U5, U6, U7, U8: symbol Comparator:LM393 -> Amp-Module-rescue:LM393-Comparator
Changed lines of the file:
@@
 TODO:\n  - Check volume impedance\n  - Check protection high level voltage\n  - Bypass caps\n  - Decide about RESERVED pins
 $Comp
-L Comparator:LM393 U4
+L Amp-Module-rescue:LM393-Comparator U4
 U 3 1 5FDE7BC8
 P 8150 4100
@@
 +5VDC
 $Comp
-L Comparator:LM393 U7
+L Amp-Module-rescue:LM393-Comparator U7
 U 1 1 5FEF8A92
 P 10350 3800
@@
 $EndComp
 $Comp
-L Comparator:LM393 U7
+L Amp-Module-rescue:LM393-Comparator U7
 U 2 1 5FEF8A98
 P 10350 4300
@@
 $EndComp
 $Comp
-L Comparator:LM393 U8
+L Amp-Module-rescue:LM393-Comparator U8
 U 2 1 5FEF8AA4
 P 10350 5300
@@
 $EndComp
 $Comp
-L Comparator:LM393 U5
+L Amp-Module-rescue:LM393-Comparator U5
 U 3 1 5FDFEC1B
 P 8150 4450
@@
 $EndComp
 $Comp
-L Comparator:LM393 U6
+L Amp-Module-rescue:LM393-Comparator U6
 U 3 1 600F6687
 P 8150 4800
@@
 $EndComp
 $Comp
-L Comparator:LM393 U7
+L Amp-Module-rescue:LM393-Comparator U7
 U 3 1 600F668D
 P 8150 5150
@@
 $EndComp
 $Comp
-L Comparator:LM393 U8
+L Amp-Module-rescue:LM393-Comparator U8
 U 3 1 60107B6A
 P 8150 5500
@@
 $EndComp
 $Comp
-L Comparator:LM393 U8
+L Amp-Module-rescue:LM393-Comparator U8
 U 1 1 5FEF8A9E
 P 10350 4800
@@
 	9900 5200 9900 5250
 $Comp
-L Comparator:LM393 U5
+L Amp-Module-rescue:LM393-Comparator U5
 U 1 1 603C66AF
 P 10350 1250
@@
 $EndComp
 $Comp
-L Comparator:LM393 U5
+L Amp-Module-rescue:LM393-Comparator U5
 U 2 1 603C66B5
 P 10350 1750
@@
 $EndComp
 $Comp
-L Comparator:LM393 U6
+L Amp-Module-rescue:LM393-Comparator U6
 U 2 1 603C66BB
 P 10350 2750
@@
 	11000 1250 11000 1750
 $Comp
-L Comparator:LM393 U6
+L Amp-Module-rescue:LM393-Comparator U6
 U 1 1 603C6712
 P 10350 2250
@@
 LM_VOUT3MON
 $Comp
-L Comparator:LM393 U4
+L Amp-Module-rescue:LM393-Comparator U4
 U 1 1 6001BFF8
 P 8600 2800
@@
 $EndComp
 $Comp
-L Comparator:LM393 U4
+L Amp-Module-rescue:LM393-Comparator U4
 U 2 1 6001CB31
 P 8600 3450
