File: KiCad/Unused.sch (KiCad schematic (older format))
At the start: 5 parts, among them U10 LM393, U11 CD4053B, U9 LM393

Commit message: updated schematic to latest KiCad version
Parts:
- U10, U9: symbol Comparator:LM393 -> Amp-Module-rescue:LM393-Comparator
Changed lines of the file:
@@
 DSP_IOUT1MON
 $Comp
-L Comparator:LM393 U?
+L Amp-Module-rescue:LM393-Comparator U?
 U 1 1 605BE17A
 P 4500 3200
@@
 $EndComp
 $Comp
-L Comparator:LM393 U?
+L Amp-Module-rescue:LM393-Comparator U?
 U 2 1 605BE180
 P 4500 3700
@@
 $EndComp
 $Comp
-L Comparator:LM393 U?
+L Amp-Module-rescue:LM393-Comparator U?
 U 1 1 605BE202
 P 4500 4200
@@
 LM_TEMPMON34
 $Comp
-L Comparator:LM393 U?
+L Amp-Module-rescue:LM393-Comparator U?
 U 3 1 605C6880
 P 8700 3200
@@
 +5VDC
 $Comp
-L Comparator:LM393 U?
+L Amp-Module-rescue:LM393-Comparator U?
 U 3 1 605C6887
 P 8700 3550
@@
 Connection ~ 8350 3450
 $Comp
-L Comparator:LM393 U?
+L Amp-Module-rescue:LM393-Comparator U?
 U 2 1 605C6F47
 P 4500 4700
